File: Corne V4 Pro Micro Edition Kicad/Corne V4 Pro Micro Edition.kicad_pcb (KiCad board)
At the start: 2 copper layers, 277.2 x 107.5 mm, 112 parts, among them J1 Conn_01x02_Socket, J2 Conn_01x02_Socket, J5 PJ-320A-DoubleSide, J6 PJ-320A-DoubleSide, SW1 SW_Push, SW10 SW_Push, SW11 SW_Push, SW12 SW_Push, SW13 SW_Push, SW14 SW_Push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

Commit message: Adding VIK Connector to support Procyon
Procyon (https://github.com/george-norton/procyon?tab=readme-ov-file) is
open-source touchpad module, the ideia is to have the option to use it
or the display on the right side, this can work with ZMK but not on
macos, QMK has full support so is a better option
Parts:
- added J3: ~, vik:vik-keyboard-connector-horizontal, F.Cu at (206.3, 118.0)
Connections:
- U1 pad 11: unconnected-(U1-P1.04-LF-Pad11) -> CHG
Routing:
- net CHG: track 0.00 -> 41.3 mm, vias 0 -> 1
- net MOSIr: track 28.1 -> 65.0 mm
- net SCKr: track 24.4 -> 54.0 mm, vias 1 -> 2
- net VCCr: track 39.7 -> 64.5 mm
- net GNDr: track 28.5 -> 53.1 mm
- removed copper zone on B.Cu, net GND
- removed copper zone on F.Cu, net GND
