File: Corne V4 Pro Micro Edition Kicad/left.kicad_sch (KiCad schematic)
At the start: 52 parts, among them J1 Conn_01x02_Socket, J1 PJ-320A-DoubleSide, SW22 PCM12SMTR, U2 Universal_Pro_Micro

Commit message: Adding VIK Connector to support Procyon
Procyon (https://github.com/george-norton/procyon?tab=readme-ov-file) is
open-source touchpad module, the ideia is to have the option to use it
or the display on the right side, this can work with ZMK but not on
macos, QMK has full support so is a better option
Parts:
- gave numbers to parts that had none: 21
- renumbered D21 to D1, D16 to D10, D10 to D11, D4 to D12, D3 to D13, D9 to D14, D14 to D16, D8 to D17, D2 to D18, D1 to D19, D18 to D2, D7 to D20, D13 to D21, D12 to D3, D6 to D4, D11 to D6, D17 to D7, D20 to D8, D19 to D9, Display1 to Display2, J1 to J6, RSW1 to RSW23, SW22 to SW44
Changed lines of the file:
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@@
 (kicad_sch
-	(version 20231120)
+	(version 20250114)
 	(generator "eeschema")
-	(generator_version "8.0")
+	(generator_version "9.0")
 	(paper "A3")
 	(title_block
@@
 		(on_board yes)
 		(dnp no)
-		(property "Reference" "D7"
+		(property "Reference" "D20"
 			(at 151.13 219.71 0)
 			(effects
@@
 		(on_board yes)
 		(dnp no)
-		(property "Reference" "SW?"
+		(property "Reference" "SW5"
 			(at 219.71 194.564 0)
 			(effects
@@
 		(on_board yes)
 		(dnp no)
-		(property "Reference" "D19"
+		(property "Reference" "D9"
 			(at 204.47 250.19 0)
 			(effects
@@
 		(dnp no)
 		(fields_autoplaced yes)
-		(property "Reference" "J1"
+		(property "Reference" "J6"
 			(at 359.7275 212.09 0)
 			(effects
@@
 		(on_board yes)
 		(dnp no)
-		(property "Reference" "SW?"
+		(property "Reference" "SW4"
 			(at 237.49 194.564 0)
 			(effects
@@
 		(on_board yes)
 		(dnp no)
-		(property "Reference" "D20"
+		(property "Reference" "D8"
 			(at 222.25 250.19 0)
 			(effects
@@
 		(on_board yes)
 		(dnp no)
-		(property "Reference" "SW?"
+		(property "Reference" "SW12"
 			(at 201.93 194.564 0)
 			(effects
@@
 		(on_board yes)
 		(dnp no)
-		(property "Reference" "SW?"
+		(property "Reference" "SW7"
 			(at 219.71 225.044 0)
 			(effects
@@
 		(on_board yes)
 		(dnp no)
-		(property "Reference" "D1"
+		(property "Reference" "D19"
 			(at 151.13 204.47 0)
 			(effects
@@
 		(on_board yes)
 		(dnp no)
-		(property "Reference" "SW?"
+		(property "Reference" "SW21"
 			(at 148.59 225.044 0)
 			(effects
@@
 		(on_board yes)
 		(dnp no)
-		(property "Reference" "D18"
+		(property "Reference" "D2"
 			(at 240.03 234.95 0)
 			(effects
@@
 		(on_board yes)
 		(dnp no)
-		(property "Reference" "SW?"
+		(property "Reference" "SW19"
 			(at 148.59 194.564 0)
 			(effects
@@
 		(on_board yes)
 		(dnp no)
-		(property "Reference" "#PWR08"
+		(property "Reference" "#PWR069"
 			(at 372.11 229.235 0)
 			(effects
@@
 		(on_board yes)
 		(dnp no)
-		(property "Reference" "SW?"
+		(property "Reference" "SW6"
 			(at 219.71 209.804 0)
 			(effects
@@
 		(on_board yes)
 		(dnp no)
-		(property "Reference" "SW?"
+		(property "Reference" "SW1"
 			(at 237.49 240.284 0)
 			(effects
@@
 		(on_board yes)
 		(dnp no)
-		(property "Reference" "SW?"
+		(property "Reference" "SW14"
 			(at 184.15 209.804 0)
 			(effects
@@
 		(on_board yes)
 		(dnp no)
-		(property "Reference" "SW?"
+		(property "Reference" "SW17"
 			(at 166.37 209.804 0)
 			(effects
@@
 		(on_board yes)
 		(dnp no)
-		(property "Reference" "D3"
+		(property "Reference" "D13"
 			(at 186.69 204.47 0)
 			(effects
@@
 		(on_board yes)
 		(dnp no)
-		(property "Reference" "D17"
+		(property "Reference" "D7"
 			(at 222.25 234.95 0)
 			(effects
@@
 		(on_board yes)
 		(dnp no)
-		(property "Reference" "#PWR05"
+		(property "Reference" "#PWR064"
 			(at 297.18 226.06 0)
 			(effects
@@
 		(on_board yes)
 		(dnp no)
-		(property "Reference" "D10"
+		(property "Reference" "D11"
 			(at 204.47 219.71 0)
 			(effects
@@
 		(on_board yes)
 		(dnp no)
-		(property "Reference" "#PWR07"
+		(property "Reference" "#PWR067"
 			(at 349.25 203.835 0)
 			(effects
@@
 		(on_board yes)
 		(dnp no)
-		(property "Reference" "D16"
+		(property "Reference" "D10"
 			(at 204.47 234.95 0)
 			(effects
@@
 		(on_board yes)
 		(dnp no)
-		(property "Reference" "SW?"
+		(property "Reference" "SW16"
 			(at 166.37 225.044 0)
 			(effects
@@
 		(on_board yes)
 		(dnp no)
-		(property "Reference" "SW?"
+		(property "Reference" "SW15"
 			(at 184.15 225.044 0)
 			(effects
@@
 		(on_board yes)
 		(dnp no)
-		(property "Reference" "SW?"
+		(property "Reference" "SW18"
 			(at 166.37 194.564 0)
 			(effects
@@
 		(on_board yes)
 		(dnp no)
-		(property "Reference" "RSW1"
+		(property "Reference" "RSW23"
 			(at 345.44 194.691 0)
 			(effects
@@
 		(on_board yes)
 		(dnp no)
-		(property "Reference" "#PWR06"
+		(property "Reference" "#PWR068"
 			(at 372.11 220.345 0)
 			(effects
@@
 		(on_board yes)
 		(dnp no)
-		(property "Reference" "#PWR019"
+		(property "Reference" "#PWR065"
 			(at 325.755 240.03 0)
 			(effects
@@
 		(on_board yes)
 		(dnp no)
-		(property "Reference" "D11"
+		(property "Reference" "D6"
 			(at 222.25 219.71 0)
 			(effects
@@
 		(on_board yes)
 		(dnp no)
-		(property "Reference" "SW?"
+		(property "Reference" "SW2"
 			(at 237.49 225.044 0)
 			(effects
@@
 		(on_board yes)
 		(dnp no)
-		(property "Reference" "D14"
+		(property "Reference" "D16"
 			(at 168.91 234.95 0)
 			(effects
@@
 		(on_board yes)
 		(dnp no)
-		(property "Reference" "D8"
+		(property "Reference" "D17"
 			(at 168.91 219.71 0)
 			(effects
@@
 		(on_board yes)
 		(dnp no)
-		(property "Reference" "D13"
+		(property "Reference" "D21"
 			(at 151.13 234.95 0)
 			(effects
@@
 		(on_board yes)
 		(dnp no)
-		(property "Reference" "#PWR03"
+		(property "Reference" "#PWR063"
 			(at 307.34 220.98 0)
 			(effects
@@
 		(on_board yes)
 		(dnp no)
-		(property "Reference" "D9"
+		(property "Reference" "D14"
 			(at 186.69 219.71 0)
 			(effects
@@
 		(on_board yes)
 		(dnp no)
-		(property "Reference" "#PWR04"
+		(property "Reference" "#PWR034"
 			(at 246.38 226.06 0)
 			(effects
@@
 		(on_board yes)
 		(dnp no)
-		(property "Reference" "D21"
+		(property "Reference" "D1"
 			(at 240.03 250.19 0)
 			(effects
@@
 		(on_board yes)
 		(dnp no)
-		(property "Reference" "SW?"
+		(property "Reference" "SW11"
 			(at 201.93 209.804 0)
 			(effects
@@
 		(on_board yes)
 		(dnp no)
-		(property "Reference" "SW?"
+		(property "Reference" "SW20"
 			(at 148.59 209.804 0)
 			(effects
@@
 		(on_board yes)
 		(dnp no)
-		(property "Reference" "SW?"
+		(property "Reference" "SW13"
 			(at 184.15 194.564 0)
 			(effects
@@
 		(on_board yes)
 		(dnp no)
-		(property "Reference" "SW?"
+		(property "Reference" "SW8"
 			(at 219.71 252.476 0)
 			(effects
@@
 		(on_board yes)
 		(dnp no)
-		(property "Reference" "D4"
+		(property "Reference" "D12"
 			(at 204.47 204.47 0)
 			(effects
@@
 		(on_board yes)
 		(dnp no)
-		(property "Reference" "#PWR018"
+		(property "Reference" "#PWR066"
 			(at 344.805 237.49 0)
 			(effects
@@
 		(on_board yes)
 		(dnp no)
-		(property "Reference" "SW?"
+		(property "Reference" "SW9"
 			(at 201.93 252.476 0)
 			(effects
@@
 		(on_board yes)
 		(dnp no)
-		(property "Reference" "D6"
+		(property "Reference" "D4"
 			(at 240.03 204.47 0)
 			(effects
@@
 		(on_board yes)
 		(dnp no)
-		(property "Reference" "SW?"
+		(property "Reference" "SW3"
 			(at 237.49 209.804 0)
 			(effects
@@
 		(on_board yes)
 		(dnp no)
-		(property "Reference" "#PWR04"
+		(property "Reference" "#PWR01"
 			(at 299.72 196.85 0)
 			(effects
@@
 		(dnp no)
 		(fields_autoplaced yes)
-		(property "Reference" "Display1"
+		(property "Reference" "Display2"
 			(at 366.395 236.22 90)
 			(effects
@@
 		(dnp no)
 		(fields_autoplaced yes)
-		(property "Reference" "SW22"
+		(property "Reference" "SW44"
 			(at 283.21 186.69 0)
 			(effects
@@
 		(on_board yes)
 		(dnp no)
-		(property "Reference" "SW?"
+		(property "Reference" "SW10"
 			(at 201.93 225.044 0)
 			(effects
@@
 		(on_board yes)
 		(dnp no)
-		(property "Reference" "D12"
+		(property "Reference" "D3"
 			(at 240.03 219.71 0)
 			(effects
@@
 		(on_board yes)
 		(dnp no)
-		(property "Reference" "D2"
+		(property "Reference" "D18"
 			(at 168.91 204.47 0)
 			(effects
