File: Corne V4 Pro Micro Edition Kicad/right.kicad_sch (KiCad schematic)
At the start: 52 parts, among them J2 Conn_01x02_Socket, J2 PJ-320A-DoubleSide, SW44 PCM12SMTR, U1 Universal_Pro_Micro

Commit message: Adding VIK Connector to support Procyon
Procyon (https://github.com/george-norton/procyon?tab=readme-ov-file) is
open-source touchpad module, the ideia is to have the option to use it
or the display on the right side, this can work with ZMK but not on
macos, QMK has full support so is a better option
Parts:
- added J3: ~, vik:vik-keyboard-connector-horizontal, symbol vik:vik-keyboard-connector
- gave numbers to parts that had none: 21
- renumbered D42 to D22, D41 to D23, D40 to D24, D39 to D25, D35 to D26, D36 to D27, D37 to D28, D38 to D29, D34 to D30, D33 to D31, D31 to D33, D28 to D34, D29 to D35, D30 to D36, D27 to D37, D26 to D38, D25 to D39, D22 to D40, D23 to D41, D24 to D42, Display2 to Display1, J2 to J5, RSW2 to RSW22, SW44 to SW43
Connections:
- net GNDr: now also J3.2 (GND)
- net MOSIr: now also J3.3 (SDA)
- net SCKr: now also J3.4 (SCL)
- net VCCr: now also J3.1 (3V3)
- net CHG: now reaches U1.11 (P1.04-LF)
- net CHG: now also J3.7 (GP_AD1)
- no-connect marks 5 -> 4
